Commit message: Modify the error code

File: src/amr_simulation/urdf/body/base.urdf.xacro (robot description, xacro)
@@ -17,5 +17,5 @@
                 <origin xyz="0 0 0.0" rpy="0 0 0" />
                 <geometry>
-                    <cylinder length="${length}" radius="${length}" />
+                    <cylinder length="${length}" radius="${radius}" />
                 </geometry>
                 <material name="white">
